File: Gowinduino.kicad_pcb (KiCad board)
At the start: 2 copper layers, 68.6 x 53.3 mm, 8 parts, among them P1 Power, P2 Analog, P3 Digital, P4 Digital, P5 CONN_01X01, P6 CONN_01X01, P7 CONN_01X01, P8 CONN_01X01

Commit message: PCB: Introduced Arduino pins.
Parts:
- added J5: SPI, Connector_PinHeader_2.54mm:PinHeader_2x03_P2.54mm_Vertical, F.Cu at (174.5, 95.9)
- J1: renamed from P1; footprint Socket_Arduino_Uno:Socket_Strip_Arduino_1x08 -> Connector_PinSocket_2.54mm:PinSocket_1x08_P2.54mm_Vertical
- J2: renamed from P2; footprint Socket_Arduino_Uno:Socket_Strip_Arduino_1x06 -> Connector_PinSocket_2.54mm:PinSocket_1x06_P2.54mm_Vertical
- J3: renamed from P3; footprint Socket_Arduino_Uno:Socket_Strip_Arduino_1x10 -> Connector_PinSocket_2.54mm:PinSocket_1x10_P2.54mm_Vertical
- J4: renamed from P4; footprint Socket_Arduino_Uno:Socket_Strip_Arduino_1x08 -> Connector_PinSocket_2.54mm:PinSocket_1x08_P2.54mm_Vertical
- turned J1 to 90 degrees
- turned J2 to 90 degrees
- turned J3 to 90 degrees
- turned J4 to 90 degrees
- renumbered P5 to PH1, P6 to PH2, P7 to PH3, P8 to PH4
Connections:
- J1 pad 1: Net-(P1-Pad1) -> (no net)
- J1 pad 2: /IOREF -> +3V3
- J1 pad 3: /Reset -> /~RESET
- J1 pad 8: /Vin -> (no net)
- J2 pad 1: /A0 -> (no net)
- J2 pad 2: /A1 -> (no net)
- J2 pad 3: /A2 -> (no net)
- J2 pad 4: /A3 -> (no net)
- J2 pad 5: /A4(SDA) -> (no net)
- J2 pad 6: /A5(SCL) -> (no net)
- J3 pad 1: /A5(SCL) -> (no net)
- J3 pad 10: /8 -> (no net)
- J3 pad 2: /A4(SDA) -> (no net)
- J3 pad 3: /AREF -> (no net)
- J3 pad 5: /13(SCK) -> (no net)
- J3 pad 6: /12(MISO) -> (no net)
- J3 pad 7: /11(**/MOSI) -> (no net)
- J3 pad 8: /10(**/SS) -> (no net)
- J3 pad 9: /9(**) -> (no net)
- J4 pad 1: /7 -> (no net)
- J4 pad 2: /6(**) -> (no net)
- J4 pad 3: /5(**) -> (no net)
- J4 pad 4: /4 -> (no net)
- J4 pad 5: /3(**) -> (no net)
- J4 pad 6: /2 -> (no net)
- J4 pad 7: /1(Tx) -> (no net)
- J4 pad 8: /0(Rx) -> (no net)
- PH1 pad 1: Net-(P5-Pad1) -> (no net)
- PH2 pad 1: Net-(P6-Pad1) -> (no net)
- PH3 pad 1: Net-(P7-Pad1) -> (no net)
- PH4 pad 1: Net-(P8-Pad1) -> (no net)
Other:
- board text removed: "1"
